Commit message: irb120 gazebo fixes

File: Learning_ROS/Part_5/irb120/irb120_description/urdf/irb120.xacro (robot description, xacro)
@@ -100,15 +100,15 @@
     <origin rpy="0 0 0" xyz="0 0 0.29"/>
     <axis xyz="0 1 0"/>
-    <limit effort="100" lower="-1.91986" upper="1.91986" velocity="4.36332"/>
+    <limit effort="500" lower="-1.91986" upper="1.91986" velocity="4.36332"/>
     <dynamics damping="1.7"/>
   </joint>
   <!-- Top Link -->
   <link name="link3">
-    <collision>
+    <!--collision>
       <origin xyz="0 0 0" rpy="0 0 0"/>
       <geometry>
 	<box size="0.2 0.2 0.2"/>
       </geometry>
-    </collision>
+    </collision-->
     <visual>
       <origin xyz="0 0 0" rpy="0 0 0"/>
@@ -129,10 +129,10 @@
   </link>
   <link name="link4">
-    <collision>
+    <!--collision>
       <origin xyz="0 0 0" rpy="0 0 0"/>
       <geometry>
 	<box size="0.2 0.2 0.2"/>
       </geometry>
-    </collision>
+    </collision-->
     <visual>
       <origin xyz="0 0 0" rpy="0 0 0"/>
@@ -164,5 +164,6 @@
       <origin xyz="0 0 0" rpy="0 0 0"/>
       <geometry>
-	<box size="0.2 0.2 0.2"/>
+	<!--box size="${width} ${width} ${height3}"/-->
+	        <mesh filename="package://irb120_description/meshes/irb120/visual/link_4.stl"/>
       </geometry>
     </collision>
@@ -193,10 +194,10 @@
   </joint>
    <link name="link6">
-    <collision>
-      <origin xyz="0 0 0" rpy="0 0 0"/>
-      <geometry>
-	<box size="0.2 0.2 0.2"/>
-      </geometry>
-    </collision>
+    <!--collision>
+      <origin xyz="0 0 0" rpy="0 0 0"/>
+      <geometry>
+	        <mesh filename="package://irb120_description/meshes/irb120/visual/link_5.stl"/>
+      </geometry>
+    </collision-->
     <visual>
       <origin xyz="0 0 0" rpy="0 0 0"/>
@@ -226,7 +227,8 @@
    <link name="link7">
     <collision>
-      <origin xyz="0 0 0" rpy="0 0 0"/>
-      <geometry>
-	<box size="0.1 0.1 0.1"/>
+     <origin xyz="0 0 0" rpy="0 0 0"/>
+      <geometry>
+	<!--box size="${width} ${width} ${height3}"/-->
+	        <mesh filename="package://irb120_description/meshes/irb120/visual/link_6.stl"/>
       </geometry>
     </collision>
